File: Home_automation.kicad_pcb (KiCad board)
At the start: 2 copper layers, 11 parts, among them Q1 BTA16-600B, Q2 BTA16-600B, Q3 BTA16-600B, Q4 BTA16-600B, Q5 BTA16-600B, Q6 BTA16-600B, U3 ESP-12E, U6 EL817, U8 AMS1117-3.3

Commit message: updated pcb
Parts:
- removed Q6: BTA16-600B, Package_TO_SOT_THT:TO-220-3_Vertical
- added C1: 10nf, Capacitor_THT:C_Rect_L13.0mm_W3.0mm_P10.00mm_FKS3_FKP3_MKS4, F.Cu at (144.2, 75.7)
- added C10: 50nf, Capacitor_THT:C_Rect_L13.0mm_W3.0mm_P10.00mm_FKS3_FKP3_MKS4, F.Cu at (115.7, 103.4)
- added C11: 10uf, Capacitor_SMD:C_0805_2012Metric, F.Cu at (166.4, 77.2)
- added C12: 1uf, Capacitor_SMD:C_0603_1608Metric_Pad1.08x0.95mm_HandSolder, F.Cu at (175.8, 86.4)
- added C13: 10nf, Capacitor_THT:C_Rect_L13.0mm_W3.0mm_P10.00mm_FKS3_FKP3_MKS4, F.Cu at (125.0, 118.8)
- added C14: 50nf, Capacitor_THT:C_Rect_L13.0mm_W3.0mm_P10.00mm_FKS3_FKP3_MKS4, F.Cu at (114.7, 127.8)
- added C2: 50nf, Capacitor_THT:C_Rect_L13.0mm_W3.0mm_P10.00mm_FKS3_FKP3_MKS4, F.Cu at (152.9, 75.8)
- added C3: 100nf, Capacitor_SMD:C_0402_1005Metric_Pad0.74x0.62mm_HandSolder, F.Cu at (187.3, 126.1)
- added C4: 100nf, Capacitor_SMD:C_0402_1005Metric_Pad0.74x0.62mm_HandSolder, F.Cu at (173.5, 107.8)
- added C5: 10nf, Capacitor_THT:C_Rect_L13.0mm_W3.0mm_P10.00mm_FKS3_FKP3_MKS4, F.Cu at (115.9, 76.6)
- added C6: 50nf, Capacitor_THT:C_Rect_L13.0mm_W3.0mm_P10.00mm_FKS3_FKP3_MKS4, F.Cu at (116.0, 85.5)
- added C7: 10nf, Capacitor_THT:C_Rect_L13.0mm_W3.0mm_P10.00mm_FKS3_FKP3_MKS4, F.Cu at (115.9, 99.4)
- added C8: 50nf, Capacitor_THT:C_Rect_L13.0mm_W3.0mm_P10.00mm_FKS3_FKP3_MKS4, F.Cu at (115.6, 89.9)
- added C9: 10nf, Capacitor_THT:C_Rect_L13.0mm_W3.0mm_P10.00mm_FKS3_FKP3_MKS4, F.Cu at (115.1, 114.0)
- added F1: Fuse, Fuse:Fuseholder_Cylinder-5x20mm_Schurter_0031_8201_Horizontal_Open, F.Cu at (211.2, 123.1)
- added JP1: SolderJumper_2_Open, my_foot:my_foot, F.Cu at (189.2, 119.5)
- added JP2: SolderJumper_2_Open, my_foot:my_foot, F.Cu at (162.3, 105.4)
- added R1: 470R, Resistor_SMD:R_0603_1608Metric_Pad0.98x0.95mm_HandSolder, F.Cu at (148.7, 86.1)
- added R10: 10K, Resistor_SMD:R_0603_1608Metric_Pad0.98x0.95mm_HandSolder, F.Cu at (190.5, 106.5)
- added R11: 470R, Resistor_SMD:R_0603_1608Metric_Pad0.98x0.95mm_HandSolder, F.Cu at (126.4, 80.8)
- added R12: 330R, Resistor_SMD:R_0603_1608Metric_Pad0.98x0.95mm_HandSolder, F.Cu at (126.4, 82.5)
- added R13: 330R, Resistor_SMD:R_0603_1608Metric_Pad0.98x0.95mm_HandSolder, F.Cu at (139.1, 80.8)
- added R14: 10K, Resistor_SMD:R_0603_1608Metric_Pad0.98x0.95mm_HandSolder, F.Cu at (202.2, 107.5)
- added R15: 39R, Resistor_SMD:R_0603_1608Metric_Pad0.98x0.95mm_HandSolder, F.Cu at (126.4, 79.3)
- added R16: 10K, Resistor_SMD:R_0603_1608Metric_Pad0.98x0.95mm_HandSolder, F.Cu at (165.3, 100.0)
- added R17: 470R, Resistor_SMD:R_0603_1608Metric_Pad0.98x0.95mm_HandSolder, F.Cu at (126.4, 94.5)
- added R18: 330R, Resistor_SMD:R_0603_1608Metric_Pad0.98x0.95mm_HandSolder, F.Cu at (126.2, 96.4)
- added R19: 330R, Resistor_SMD:R_0603_1608Metric_Pad0.98x0.95mm_HandSolder, F.Cu at (139.1, 95.6)
- added R2: 330R, Resistor_SMD:R_0603_1608Metric_Pad0.98x0.95mm_HandSolder, F.Cu at (150.3, 86.1)
- added R20: 47K, Resistor_SMD:R_0603_1608Metric_Pad0.98x0.95mm_HandSolder, F.Cu at (184.5, 129.4)
- added R21: 39R, Resistor_SMD:R_0603_1608Metric_Pad0.98x0.95mm_HandSolder, F.Cu at (126.3, 92.7)
- added R22: 2K, Resistor_SMD:R_0603_1608Metric_Pad0.98x0.95mm_HandSolder, F.Cu at (188.7, 103.2)
- added R23: 47K, Resistor_SMD:R_0603_1608Metric_Pad0.98x0.95mm_HandSolder, F.Cu at (204.9, 116.6)
- added R24: 470R, Resistor_SMD:R_0603_1608Metric_Pad0.98x0.95mm_HandSolder, F.Cu at (125.1, 109.1)
- added R25: 330R, Resistor_SMD:R_0603_1608Metric_Pad0.98x0.95mm_HandSolder, F.Cu at (125.2, 110.9)
- added R26: 330R, Resistor_SMD:R_0603_1608Metric_Pad0.98x0.95mm_HandSolder, F.Cu at (138.2, 110.0)
- added R27: 39R, Resistor_SMD:R_0603_1608Metric_Pad0.98x0.95mm_HandSolder, F.Cu at (125.4, 107.0)
- added R28: 10K, Resistor_SMD:R_0603_1608Metric_Pad0.98x0.95mm_HandSolder, F.Cu at (190.9, 99.5)
- added R29: 10K, Resistor_SMD:R_0603_1608Metric_Pad0.98x0.95mm_HandSolder, F.Cu at (170.0, 99.4)
- added R3: 330R, Resistor_SMD:R_0603_1608Metric_Pad0.98x0.95mm_HandSolder, F.Cu at (148.1, 98.7)
- added R30: 470R, Resistor_SMD:R_0603_1608Metric_Pad0.98x0.95mm_HandSolder, F.Cu at (125.5, 123.4)
- added R31: 330R, Resistor_SMD:R_0603_1608Metric_Pad0.98x0.95mm_HandSolder, F.Cu at (125.6, 125.3)
- added R32: 330R, Resistor_SMD:R_0603_1608Metric_Pad0.98x0.95mm_HandSolder, F.Cu at (138.5, 125.1)
- added R33: 39R, Resistor_SMD:R_0603_1608Metric_Pad0.98x0.95mm_HandSolder, F.Cu at (125.7, 121.5)
- added R34: 10K, Resistor_SMD:R_0603_1608Metric_Pad0.98x0.95mm_HandSolder, F.Cu at (183.1, 97.5)
- added R35: 10K, Resistor_SMD:R_0603_1608Metric_Pad0.98x0.95mm_HandSolder, F.Cu at (174.4, 97.7)
- added R36: 10K, Resistor_SMD:R_0603_1608Metric_Pad0.98x0.95mm_HandSolder, F.Cu at (187.3, 99.3)
- added R4: 39R, Resistor_SMD:R_0603_1608Metric_Pad0.98x0.95mm_HandSolder, F.Cu at (147.0, 86.1)
- added R5: 10K, Resistor_SMD:R_0603_1608Metric_Pad0.98x0.95mm_HandSolder, F.Cu at (175.6, 129.5)
- added R6: 10K, Resistor_SMD:R_0603_1608Metric_Pad0.98x0.95mm_HandSolder, F.Cu at (180.9, 128.9)
- added R7: 10K, Resistor_SMD:R_0603_1608Metric_Pad0.98x0.95mm_HandSolder, F.Cu at (188.3, 109.6)
- added R8: 10K, Resistor_SMD:R_0603_1608Metric_Pad0.98x0.95mm_HandSolder, F.Cu at (178.8, 97.2)
- added R9: 10K, Resistor_SMD:R_0603_1608Metric_Pad0.98x0.95mm_HandSolder, F.Cu at (165.5, 102.9)
- added TP1: TestPoint, TestPoint:TestPoint_Loop_D3.80mm_Drill2.0mm, F.Cu at (147.6, 71.4)
- added TP10: TestPoint, TestPoint:TestPoint_Pad_1.0x1.0mm, F.Cu at (165.6, 95.6)
- added TP11: TestPoint, TestPoint:TestPoint_Pad_1.0x1.0mm, F.Cu at (167.3, 85.0)
- added TP12: TestPoint, TestPoint:TestPoint_Pad_1.0x1.0mm, F.Cu at (167.3, 88.1)
- added TP13: TestPoint, TestPoint:TestPoint_Pad_1.0x1.0mm, F.Cu at (167.3, 91.1)
- added TP14: TestPoint, TestPoint:TestPoint_Loop_D3.80mm_Drill2.0mm, F.Cu at (110.1, 108.8)
- added TP15: TestPoint, TestPoint:TestPoint_Loop_D3.80mm_Drill2.0mm, F.Cu at (219.6, 83.0)
- added TP17: TestPoint, TestPoint:TestPoint_Loop_D3.80mm_Drill2.0mm, F.Cu at (218.9, 76.5)
- added TP18: TestPoint, TestPoint:TestPoint_Loop_D3.80mm_Drill2.0mm, F.Cu at (196.5, 97.6)
- added TP19: TestPoint, TestPoint:TestPoint_Loop_D3.80mm_Drill2.0mm, F.Cu at (196.5, 103.3)
- added TP20: TestPoint, TestPoint:TestPoint_Loop_D3.80mm_Drill2.0mm, F.Cu at (228.1, 95.4)
- added TP21: TestPoint, TestPoint:TestPoint_Loop_D3.80mm_Drill2.0mm, F.Cu at (110.5, 123.8)
- added TP22: TestPoint, TestPoint:TestPoint_Loop_D3.80mm_Drill2.0mm, F.Cu at (196.5, 108.9)
- added TP23: TestPoint, TestPoint:TestPoint_Loop_D3.80mm_Drill2.0mm, F.Cu at (228.1, 101.1)
- added TP24: TestPoint, TestPoint:TestPoint_Loop_D3.80mm_Drill2.0mm, F.Cu at (228.1, 106.7)
- added TP26: TestPoint, TestPoint:TestPoint_Loop_D3.80mm_Drill2.0mm, F.Cu at (228.1, 112.4)
- added TP3: TestPoint, TestPoint:TestPoint_Pad_1.0x1.0mm, F.Cu at (164.2, 85.0)
- added TP4: TestPoint, TestPoint:TestPoint_Loop_D3.80mm_Drill2.0mm, F.Cu at (111.0, 80.7)
- added TP6: TestPoint, TestPoint:TestPoint_Loop_D3.80mm_Drill2.0mm, F.Cu at (110.1, 95.2)
- added TP8: TestPoint, TestPoint:TestPoint_Pad_1.0x1.0mm, F.Cu at (164.2, 88.1)
- added TP9: TestPoint, TestPoint:TestPoint_Pad_1.0x1.0mm, F.Cu at (164.2, 91.1)
- added U1: MOC3010M, Package_DIP:DIP-6_W7.62mm, F.Cu at (148.1, 96.6)
- added U2: MOC3010M, Package_DIP:DIP-6_W7.62mm, F.Cu at (137.1, 81.7)
- added U4: MOC3010M, Package_DIP:DIP-6_W7.62mm, F.Cu at (137.0, 96.4)
- added U7: AMS1117-3.3, Package_TO_SOT_SMD:SOT-223-3_TabPin2, F.Cu at (173.3, 77.8)
- added U9: EL817, Package_DIP:DIP-4_W7.62mm, F.Cu at (190.5, 123.2)
- U6: value EL817 -> MOC3010M; footprint Package_DIP:DIP-4_W7.62mm -> Package_DIP:DIP-6_W7.62mm
- U8: value AMS1117-3.3 -> MOC3010M; footprint Package_TO_SOT_SMD:SOT-223-3_TabPin2 -> Package_DIP:DIP-6_W7.62mm
- moved PS1 57.6 mm to (197.0, 79.1), turned to 180 degrees
- moved U8 48.9 mm to (136.3, 126.2), turned to 180 degrees
- moved D1 47.6 mm to (199.7, 117.0)
- moved U3 33.1 mm to (158.8, 119.1), turned to 180 degrees
- moved U6 28.8 mm to (136.1, 111.1), turned to 180 degrees
- moved Q1 23.9 mm to (147.6, 76.5), turned to -90 degrees
- moved Q5 20.6 mm to (115.8, 124.2)
- moved Q4 13.6 mm to (115.2, 109.7)
- moved Q2 9.41 mm to (116.8, 81.9)
- moved Q3 8.76 mm to (115.9, 95.8)
Connections:
- PS1 pad 1: Net-(PS1-AC1) -> AC
- U3 pad 10: IO2 -> S2
- U3 pad 12: S1 -> S4
- U3 pad 13: IO3 -> S5
- U3 pad 14: IO3 -> Zero_C
- U3 pad 4: S2 -> S1
- U3 pad 5: S4 -> P5
- U6 pad 1: Net-(D1-Pad1) -> Net-(R26-Pad2)
- U6 pad 2: Net-(D1-Pad3) -> GND
- U6 pad 3: Net-(R25-Pad1) -> unconnected-(U6-NC-Pad3)
- U6 pad 4: Zero_C -> Net-(Q4-G)
- U8 pad 1: GND -> Net-(R32-Pad2)
- U8 pad 2: 3v3 -> GND
- U8 pad 3: Vcc -> unconnected-(U8-NC-Pad3)

Commit message: Add files via upload
made pcb
Parts:
- TP18, TP19, TP20, TP22, TP23, TP24: footprint TestPoint:TestPoint_Loop_D3.80mm_Drill2.0mm -> TestPoint:TestPoint_THTPad_D2.0mm_Drill1.0mm
- moved TP21 103.0 mm to (201.3, 75.1), turned to -90 degrees
- moved TP26 96.3 mm to (139.1, 75.5), turned to 90 degrees
- moved TP4 96.1 mm to (201.9, 112.1), turned to 180 degrees
- moved C14 95.5 mm to (197.0, 79.4), turned to 180 degrees
- moved Q5 94.6 mm to (196.0, 74.1), turned to 180 degrees
- moved TP14 94.2 mm to (201.7, 86.9), turned to 180 degrees
- moved TP23 93.8 mm to (138.5, 128.7)
- moved TP6 92.0 mm to (202.0, 99.2), turned to 180 degrees
- moved TP20 91.3 mm to (138.6, 113.3)
- moved TP24 90.1 mm to (138.6, 116.5)
- moved R33 89.7 mm to (199.6, 70.7), turned to -90 degrees
- moved C9 87.6 mm to (197.1, 83.1), turned to 180 degrees
- moved C5 87.4 mm to (197.3, 108.4), turned to 180 degrees
- moved C6 87.3 mm to (197.4, 117.1), turned to 180 degrees
- moved C13 86.6 mm to (197.0, 70.8)
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Connections:
- U3 pad 10: S2 -> S1
- U3 pad 11: S3 -> S2
- U3 pad 12: S4 -> S3
- U3 pad 13: S5 -> S4
- U3 pad 14: Zero_C -> S5
- U3 pad 19: P1 -> Zero_C
- U3 pad 20: P2 -> IO1
- U3 pad 4: S1 -> P1
- U3 pad 5: P5 -> P2
- U3 pad 9: IO1 -> P5
Routing:
- net GNDPWR: track 0.00 -> 190.5 mm, vias 0 -> 1
- net 3v3: track 0.00 -> 65.1 mm, vias 0 -> 4
- net AC: track 0.00 -> 55.2 mm
- net S1: track 0.00 -> 38.2 mm, vias 0 -> 1
- net S2: track 0.00 -> 36.4 mm, vias 0 -> 1
- net GND: track 0.00 -> 33.9 mm, vias 0 -> 4
- net Net-(R32-Pad2): track 0.00 -> 32.8 mm
- net S3: track 0.00 -> 32.3 mm, vias 0 -> 1
- net S4: track 0.00 -> 29.5 mm, vias 0 -> 1
- net S5: track 0.00 -> 28.9 mm, vias 0 -> 1
- net Net-(R26-Pad2): track 0.00 -> 27.4 mm
- net Net-(Q3-A1): track 0.00 -> 21.2 mm
- net Net-(Q1-A1): track 0.00 -> 21.1 mm
- net Net-(Q5-A1): track 0.00 -> 21.1 mm
- net Net-(Q2-A1): track 0.00 -> 20.5 mm
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- added copper zone on B.Cu, net GND
- added copper zone on F.Cu, net GND
- added copper zone on B.Cu, net GNDPWR
- added copper zone on F.Cu, net GNDPWR
Other:
- board outline added: 71.4 x 66.2 mm
